Commit message: Sync envs/ from fede master (the env Tom's demos were collected on)
Replaces envs/place.py, base_random_env.py, robot/so101.urdf and adds
meshes/bowl_carton.obj with the versions from fedecomi04/squint master.
This is the exact environment the synthetic FK/IK demos
(scripts/collect_rlpd_demos.py / Tom's tom-separating-cubes pipeline)
were generated on, so RLPD training with --offline_path now matches the
demo-collection env (controller, scene, bowl mesh, robot URDF, DR/camera
config in base_random_env).

Notable: fede master is AHEAD of our fork on:
  - base_random_env.py (+96 lines: newer DR / camera / lighting)
  - place.py split-mode work (split_closest_first, split_low_hover_*)
  - so101.urdf (+29 lines, updated robot geometry)
  - meshes/bowl_carton.obj (new bowl mesh)

Lost vs our previous place.py (recoverable via git history at ab40af2):
  - skip_bowl flag and its gating
  - squint_native_reward function and reward shaping experiments

train_rlpd.py / train_squint.py: skip_bowl and squint_native_reward are
now passed to the env ONLY when True (they don't exist in fede master's
place.py), so a standard run doesn't hit an unexpected-kwarg TypeError.
Enabling either again requires re-adding the flag to place.py.

Co-Authored-By: Claude Opus 4.7 (1M context) <noreply@anthropic.com>

File: envs/robot/so101.urdf (robot description, URDF)
Before this commit: robot so101, 10 links, 9 joints
Links:
- added link camera_shadow_box, mass 1e-6; visual box size=0.03 0.03 0.03
Joints:
- added joint camera_shadow_joint: type fixed, parent gripper_link, child camera_shadow_box, origin xyz=-0.0006 0.0498 -0.033 rpy=0 0 0
